Commit message: feat(urdf): add REV00 CAD inertial properties

File: 03_CAD/URDF/matt_robodog_rev00/matt_robodog_rev00.urdf (robot description, URDF)
Before this commit: robot matt_robodog_rev00, 17 links, 16 joints
Links:
- link base_link: mass None -> 1.282000
- link lf_foot_link: mass None -> 0.017500
- link lf_hip_link: mass None -> 0.050000
- link lf_lower_leg_link: mass None -> 0.059500
- link lf_upper_leg_link: mass None -> 0.172500
- link lh_foot_link: mass None -> 0.017500
- link lh_hip_link: mass None -> 0.050000
- link lh_lower_leg_link: mass None -> 0.059500
- link lh_upper_leg_link: mass None -> 0.172500
- link rf_foot_link: mass None -> 0.017500
- link rf_hip_link: mass None -> 0.050000
- link rf_lower_leg_link: mass None -> 0.059500
- link rf_upper_leg_link: mass None -> 0.172500
- link rh_foot_link: mass None -> 0.017500
- link rh_hip_link: mass None -> 0.050000
- link rh_lower_leg_link: mass None -> 0.059500
- link rh_upper_leg_link: mass None -> 0.172500

Commit message: fix(urdf): declare STL millimetre mesh scale

File: 03_CAD/URDF/matt_robodog_rev00/matt_robodog_rev00.urdf (robot description, URDF)
Before this commit: robot matt_robodog_rev00, 17 links, 16 joints
Links:
- link base_link: geometry collision mesh filename=meshes/base_link.stl scale=0.001 0.001 0.001; visual mesh filename=meshes/base_link.stl scale=0.001 0.001 0.001
- link lf_foot_link: geometry collision mesh filename=meshes/lf_foot_link.stl scale=0.001 0.001 0.001; visual mesh filename=meshes/lf_foot_link.stl scale=0.001 0.001 0.001
- link lf_hip_link: geometry collision mesh filename=meshes/lf_hip_link.stl scale=0.001 0.001 0.001; visual mesh filename=meshes/lf_hip_link.stl scale=0.001 0.001 0.001
- link lf_lower_leg_link: geometry collision mesh filename=meshes/lf_lower_leg_link.stl scale=0.001 0.001 0.001; visual mesh filename=meshes/lf_lower_leg_link.stl scale=0.001 0.001 0.001
- link lf_upper_leg_link: geometry collision mesh filename=meshes/lf_upper_leg_link.stl scale=0.001 0.001 0.001; visual mesh filename=meshes/lf_upper_leg_link.stl scale=0.001 0.001 0.001
- link lh_foot_link: geometry collision mesh filename=meshes/lh_foot_link.stl scale=0.001 0.001 0.001; visual mesh filename=meshes/lh_foot_link.stl scale=0.001 0.001 0.001
- link lh_hip_link: geometry collision mesh filename=meshes/lh_hip_link.stl scale=0.001 0.001 0.001; visual mesh filename=meshes/lh_hip_link.stl scale=0.001 0.001 0.001
- link lh_lower_leg_link: geometry collision mesh filename=meshes/lh_lower_leg_link.stl scale=0.001 0.001 0.001; visual mesh filename=meshes/lh_lower_leg_link.stl scale=0.001 0.001 0.001
- link lh_upper_leg_link: geometry collision mesh filename=meshes/lh_upper_leg_link.stl scale=0.001 0.001 0.001; visual mesh filename=meshes/lh_upper_leg_link.stl scale=0.001 0.001 0.001
- link rf_foot_link: geometry collision mesh filename=meshes/rf_foot_link.stl scale=0.001 0.001 0.001; visual mesh filename=meshes/rf_foot_link.stl scale=0.001 0.001 0.001
- link rf_hip_link: geometry collision mesh filename=meshes/rf_hip_link.stl scale=0.001 0.001 0.001; visual mesh filename=meshes/rf_hip_link.stl scale=0.001 0.001 0.001
- link rf_lower_leg_link: geometry collision mesh filename=meshes/rf_lower_leg_link.stl scale=0.001 0.001 0.001; visual mesh filename=meshes/rf_lower_leg_link.stl scale=0.001 0.001 0.001
- link rf_upper_leg_link: geometry collision mesh filename=meshes/rf_upper_leg_link.stl scale=0.001 0.001 0.001; visual mesh filename=meshes/rf_upper_leg_link.stl scale=0.001 0.001 0.001
- link rh_foot_link: geometry collision mesh filename=meshes/rh_foot_link.stl scale=0.001 0.001 0.001; visual mesh filename=meshes/rh_foot_link.stl scale=0.001 0.001 0.001
- link rh_hip_link: geometry collision mesh filename=meshes/rh_hip_link.stl scale=0.001 0.001 0.001; visual mesh filename=meshes/rh_hip_link.stl scale=0.001 0.001 0.001
- link rh_lower_leg_link: geometry collision mesh filename=meshes/rh_lower_leg_link.stl scale=0.001 0.001 0.001; visual mesh filename=meshes/rh_lower_leg_link.stl scale=0.001 0.001 0.001
- link rh_upper_leg_link: geometry collision mesh filename=meshes/rh_upper_leg_link.stl scale=0.001 0.001 0.001; visual mesh filename=meshes/rh_upper_leg_link.stl scale=0.001 0.001 0.001
Joints:
- joint lf_lower_leg_joint: limit lower=-1.6057029118347832 upper=0.654498469498 effort=0.902244 velocity=3.03687289847 -> lower=-1.701696020690 upper=0.654498469498 effort=0.902244 velocity=3.03687289847
- joint lh_lower_leg_joint: limit lower=-1.6057029118347832 upper=0.654498469498 effort=0.902244 velocity=3.03687289847 -> lower=-1.701696020690 upper=0.654498469498 effort=0.902244 velocity=3.03687289847
- joint rf_lower_leg_joint: limit lower=-1.6057029118347832 upper=0.654498469498 effort=0.902244 velocity=3.03687289847 -> lower=-1.701696020690 upper=0.654498469498 effort=0.902244 velocity=3.03687289847
- joint rh_lower_leg_joint: limit lower=-1.6057029118347832 upper=0.654498469498 effort=0.902244 velocity=3.03687289847 -> lower=-1.701696020690 upper=0.654498469498 effort=0.902244 velocity=3.03687289847

Commit message: fix(matdog): sync lower-leg limits and calibration references

File: 03_CAD/URDF/matt_robodog_rev00/matt_robodog_rev00.urdf (robot description, URDF)
Before this commit: robot matt_robodog_rev00, 17 links, 16 joints
Joints:
- joint lf_lower_leg_joint: limit lower=-1.701696020690 upper=0.654498469498 effort=0.902244 velocity=3.03687289847 -> lower=-1.605702911835 upper=0.654498469498 effort=0.902244 velocity=3.03687289847
- joint lh_lower_leg_joint: limit lower=-1.701696020690 upper=0.654498469498 effort=0.902244 velocity=3.03687289847 -> lower=-1.605702911835 upper=0.654498469498 effort=0.902244 velocity=3.03687289847
- joint rf_lower_leg_joint: limit lower=-1.701696020690 upper=0.654498469498 effort=0.902244 velocity=3.03687289847 -> lower=-1.605702911835 upper=0.654498469498 effort=0.902244 velocity=3.03687289847
- joint rh_lower_leg_joint: limit lower=-1.701696020690 upper=0.654498469498 effort=0.902244 velocity=3.03687289847 -> lower=-1.605702911835 upper=0.654498469498 effort=0.902244 velocity=3.03687289847

Commit message: add deterministic Geometry Compiler V5

File: 03_CAD/URDF/matt_robodog_rev00/matt_robodog_rev00.urdf (robot description, URDF)
Before this commit: robot matt_robodog_rev00, 17 links, 16 joints
Links:
- link base_link: geometry collision mesh filename=meshes/collision/base_link.stl scale=0.001 0.001 0.001; visual mesh filename=meshes/base_link.stl scale=0.001 0.001 0.001
- link lf_foot_link: geometry collision mesh filename=meshes/collision/lf_foot_link.stl scale=0.001 0.001 0.001; visual mesh filename=meshes/lf_foot_link.stl scale=0.001 0.001 0.001
- link lf_hip_link: geometry collision mesh filename=meshes/collision/lf_hip_link.stl scale=0.001 0.001 0.001; visual mesh filename=meshes/lf_hip_link.stl scale=0.001 0.001 0.001
- link lf_lower_leg_link: geometry collision mesh filename=meshes/collision/lf_lower_leg_link.stl scale=0.001 0.001 0.001; visual mesh filename=meshes/lf_lower_leg_link.stl scale=0.001 0.001 0.001
- link lf_upper_leg_link: geometry collision mesh filename=meshes/collision/lf_upper_leg_link.stl scale=0.001 0.001 0.001; visual mesh filename=meshes/lf_upper_leg_link.stl scale=0.001 0.001 0.001
- link lh_foot_link: geometry collision mesh filename=meshes/collision/lh_foot_link.stl scale=0.001 0.001 0.001; visual mesh filename=meshes/lh_foot_link.stl scale=0.001 0.001 0.001
- link lh_hip_link: geometry collision mesh filename=meshes/collision/lh_hip_link.stl scale=0.001 0.001 0.001; visual mesh filename=meshes/lh_hip_link.stl scale=0.001 0.001 0.001
- link lh_lower_leg_link: geometry collision mesh filename=meshes/collision/lh_lower_leg_link.stl scale=0.001 0.001 0.001; visual mesh filename=meshes/lh_lower_leg_link.stl scale=0.001 0.001 0.001
- link lh_upper_leg_link: geometry collision mesh filename=meshes/collision/lh_upper_leg_link.stl scale=0.001 0.001 0.001; visual mesh filename=meshes/lh_upper_leg_link.stl scale=0.001 0.001 0.001
- link rf_foot_link: geometry collision mesh filename=meshes/collision/rf_foot_link.stl scale=0.001 0.001 0.001; visual mesh filename=meshes/rf_foot_link.stl scale=0.001 0.001 0.001
- link rf_hip_link: geometry collision mesh filename=meshes/collision/rf_hip_link.stl scale=0.001 0.001 0.001; visual mesh filename=meshes/rf_hip_link.stl scale=0.001 0.001 0.001
- link rf_lower_leg_link: geometry collision mesh filename=meshes/collision/rf_lower_leg_link.stl scale=0.001 0.001 0.001; visual mesh filename=meshes/rf_lower_leg_link.stl scale=0.001 0.001 0.001
- link rf_upper_leg_link: geometry collision mesh filename=meshes/collision/rf_upper_leg_link.stl scale=0.001 0.001 0.001; visual mesh filename=meshes/rf_upper_leg_link.stl scale=0.001 0.001 0.001
- link rh_foot_link: geometry collision mesh filename=meshes/collision/rh_foot_link.stl scale=0.001 0.001 0.001; visual mesh filename=meshes/rh_foot_link.stl scale=0.001 0.001 0.001
- link rh_hip_link: geometry collision mesh filename=meshes/collision/rh_hip_link.stl scale=0.001 0.001 0.001; visual mesh filename=meshes/rh_hip_link.stl scale=0.001 0.001 0.001
- link rh_lower_leg_link: geometry collision mesh filename=meshes/collision/rh_lower_leg_link.stl scale=0.001 0.001 0.001; visual mesh filename=meshes/rh_lower_leg_link.stl scale=0.001 0.001 0.001
- link rh_upper_leg_link: geometry collision mesh filename=meshes/collision/rh_upper_leg_link.stl scale=0.001 0.001 0.001; visual mesh filename=meshes/rh_upper_leg_link.stl scale=0.001 0.001 0.001
