Commit message: geometry: integrate REV01-FIX base_link and HIP +2.2 mm; unify visual/collision meshes
Validated offline with the unmodified Geometry Compiler V5: q=0 12/12 pairs
separated, 24/24 endpoint searches, no new collision or regression vs REV00
(22 endpoints identical; two hip endpoints move 6.8e-5 rad, below the 1e-4
bisection resolution). Pin/socket clearance measured on the STL meshes.

- base_link collision mesh = REV01-FIX (sha256 c2eadf63..., 36832 triangles)
- four hip_joint origins +2.2 mm in Z (LF/RF 0.0487, RH/LH 0.0287)
- every <visual> uses the same meshes/collision/<link>.stl as <collision>;
  the 17 decorative STL under meshes/ are removed (recoverable from history)
- LegGeometryData.h regenerated with matdog_motion_geometry_export.py
- URDF/FK/stance/foot-contact/manifest/immutability pins and affected tests
  updated; FK/IK and viewer verified against the new model
- evidence in 09_Logs/Validation_Reports/REV01_FIX_Integration_2026-10-30

Not changed: calibrations, NVS, servo offsets, mechanical limits, V5 kernel,
installed firmware. The firmware calibration chain (Calibration*Data.h,
MATDOG_JOINT_CALIBRATION.yaml) is still bound to the REV00 URDF hash and
fails static_audit until its provenance is decided; see REPORT.md.

Co-Authored-By: Claude Sonnet 5.5 <noreply@anthropic.com>

File: 03_CAD/URDF/matt_robodog_rev00/matt_robodog_rev00.urdf (robot description, URDF)
Before this commit: robot matt_robodog_rev00, 17 links, 16 joints
Links:
- link base_link: geometry collision mesh filename=meshes/collision/base_link.stl scale=0.001 0.001 0.001; visual mesh filename=meshes/collision/base_link.stl scale=0.001 0.001 0.001
- link lf_foot_link: geometry collision mesh filename=meshes/collision/lf_foot_link.stl scale=0.001 0.001 0.001; visual mesh filename=meshes/collision/lf_foot_link.stl scale=0.001 0.001 0.001
- link lf_hip_link: geometry collision mesh filename=meshes/collision/lf_hip_link.stl scale=0.001 0.001 0.001; visual mesh filename=meshes/collision/lf_hip_link.stl scale=0.001 0.001 0.001
- link lf_lower_leg_link: geometry collision mesh filename=meshes/collision/lf_lower_leg_link.stl scale=0.001 0.001 0.001; visual mesh filename=meshes/collision/lf_lower_leg_link.stl scale=0.001 0.001 0.001
- link lf_upper_leg_link: geometry collision mesh filename=meshes/collision/lf_upper_leg_link.stl scale=0.001 0.001 0.001; visual mesh filename=meshes/collision/lf_upper_leg_link.stl scale=0.001 0.001 0.001
- link lh_foot_link: geometry collision mesh filename=meshes/collision/lh_foot_link.stl scale=0.001 0.001 0.001; visual mesh filename=meshes/collision/lh_foot_link.stl scale=0.001 0.001 0.001
- link lh_hip_link: geometry collision mesh filename=meshes/collision/lh_hip_link.stl scale=0.001 0.001 0.001; visual mesh filename=meshes/collision/lh_hip_link.stl scale=0.001 0.001 0.001
- link lh_lower_leg_link: geometry collision mesh filename=meshes/collision/lh_lower_leg_link.stl scale=0.001 0.001 0.001; visual mesh filename=meshes/collision/lh_lower_leg_link.stl scale=0.001 0.001 0.001
- link lh_upper_leg_link: geometry collision mesh filename=meshes/collision/lh_upper_leg_link.stl scale=0.001 0.001 0.001; visual mesh filename=meshes/collision/lh_upper_leg_link.stl scale=0.001 0.001 0.001
- link rf_foot_link: geometry collision mesh filename=meshes/collision/rf_foot_link.stl scale=0.001 0.001 0.001; visual mesh filename=meshes/collision/rf_foot_link.stl scale=0.001 0.001 0.001
- link rf_hip_link: geometry collision mesh filename=meshes/collision/rf_hip_link.stl scale=0.001 0.001 0.001; visual mesh filename=meshes/collision/rf_hip_link.stl scale=0.001 0.001 0.001
- link rf_lower_leg_link: geometry collision mesh filename=meshes/collision/rf_lower_leg_link.stl scale=0.001 0.001 0.001; visual mesh filename=meshes/collision/rf_lower_leg_link.stl scale=0.001 0.001 0.001
- link rf_upper_leg_link: geometry collision mesh filename=meshes/collision/rf_upper_leg_link.stl scale=0.001 0.001 0.001; visual mesh filename=meshes/collision/rf_upper_leg_link.stl scale=0.001 0.001 0.001
- link rh_foot_link: geometry collision mesh filename=meshes/collision/rh_foot_link.stl scale=0.001 0.001 0.001; visual mesh filename=meshes/collision/rh_foot_link.stl scale=0.001 0.001 0.001
- link rh_hip_link: geometry collision mesh filename=meshes/collision/rh_hip_link.stl scale=0.001 0.001 0.001; visual mesh filename=meshes/collision/rh_hip_link.stl scale=0.001 0.001 0.001
- link rh_lower_leg_link: geometry collision mesh filename=meshes/collision/rh_lower_leg_link.stl scale=0.001 0.001 0.001; visual mesh filename=meshes/collision/rh_lower_leg_link.stl scale=0.001 0.001 0.001
- link rh_upper_leg_link: geometry collision mesh filename=meshes/collision/rh_upper_leg_link.stl scale=0.001 0.001 0.001; visual mesh filename=meshes/collision/rh_upper_leg_link.stl scale=0.001 0.001 0.001
Joints:
- joint lf_hip_joint: origin xyz=0.1125 0.0475 0.0465 rpy=0 0 0 -> xyz=0.1125 0.0475 0.0487 rpy=0 0 0
- joint lh_hip_joint: origin xyz=-0.1125 0.0475 0.0265 rpy=0 0 0 -> xyz=-0.1125 0.0475 0.0287 rpy=0 0 0
- joint rf_hip_joint: origin xyz=0.1125 -0.0475 0.0465 rpy=0 0 0 -> xyz=0.1125 -0.0475 0.0487 rpy=0 0 0
- joint rh_hip_joint: origin xyz=-0.1125 -0.0475 0.0265 rpy=0 0 0 -> xyz=-0.1125 -0.0475 0.0287 rpy=0 0 0

Commit message: physical properties: Solid Edge 2026-10-30 inertials for the 17 links, single workbook, calibration-basis delta
- URDF: only the 17 <inertial> blocks change (masses, CoM, tensors rebuilt at the CoM from principal
  axes + radii of gyration). Nominal configuration includes the Jetson Orin (in the CAD); the
  2.807 kg weighing (no Jetson) is historical evidence. Everything except <inertial> is
  canonically identical (digest d66fa1cc...); no STL, joint, limit, HIP or calibration file changes.
- Reconciliation: 17 links 2.928 kg vs Solid Edge assembly 2.937 kg; volumes close within 1.1 mm3,
  the 9 g residual is at the 1 g report resolution and is neither allocated nor scaled.
- matdog_calibration_basis.py: the declared delta now also admits the 17 <inertial> blocks, with
  structural and physical checks; any other change still fails. Basis files, hashes, tag
  3713f4ddc43b204e and the gen-1 chain are untouched.
- Derived data refreshed with the existing tools: model manifest, LegGeometryData.h (only
  kUrdfSha256 changes), pins and tests that follow the operational URDF.
- Workbook Coordinate_Cinematiche_matt_robodog_rev00.xlsx updated in place (formulas kept, masses
  read from Inertial_Properties, HIP Z 48.7/28.7 mm, unified mesh paths, weight evidence sheet);
  history is kept by Git.
- Evidence, tools and report in 09_Logs/Validation_Reports/REV01_FIX_Physical_Properties_2026-10-31/.

Offline only; no dynamic hardware validation. No flash, q0 capture, calibration, NVS or EEPROM access.

Co-Authored-By: Claude Sonnet 5.5 <noreply@anthropic.com>

File: 03_CAD/URDF/matt_robodog_rev00/matt_robodog_rev00.urdf (robot description, URDF)
Before this commit: robot matt_robodog_rev00, 17 links, 16 joints
Links:
- link base_link: mass 1.282000 -> 1.828000
- link lf_foot_link: mass 0.017500 -> 0.014000
- link lf_lower_leg_link: mass 0.059500 -> 0.059000
- link lf_upper_leg_link: mass 0.172500 -> 0.152000
- link lh_foot_link: mass 0.017500 -> 0.014000
- link lh_lower_leg_link: mass 0.059500 -> 0.059000
- link lh_upper_leg_link: mass 0.172500 -> 0.152000
- link rf_foot_link: mass 0.017500 -> 0.014000
- link rf_lower_leg_link: mass 0.059500 -> 0.059000
- link rf_upper_leg_link: mass 0.172500 -> 0.152000
- link rh_foot_link: mass 0.017500 -> 0.014000
- link rh_lower_leg_link: mass 0.059500 -> 0.059000
- link rh_upper_leg_link: mass 0.172500 -> 0.152000
